File: Hardware/Qwiic_RTC_RV8803.brd (EAGLE design)
At the start: 25.4 x 25.4 mm, 49 parts, among them J1 QWIIC, J2 QWIIC, U1 RV-8803

Commit message: Updating silk
Parts:
- moved U$22 8.89 mm to (17.0, 8.21)
- moved U$21 8.89 mm to (17.0, 9.51)
- moved LOGO1 8.57 mm to (12.7, 12.0)
Changed lines of the file:
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@@
 <element name="U$16" library="buzzard_labels" package="#INT5" value="" x="16.51" y="1.397" smashed="yes" rot="MR90"/>
 <element name="U$17" library="buzzard_labels (1)" package="PWR7" value="" x="1.27" y="3.302" smashed="yes" rot="R90"/>
-<element name="LOGO1" library="SparkFun-Aesthetics" package="SFE_LOGO_NAME_FLAME_.1" value="SFE_LOGO_NAME_FLAME.1_INCH" x="12.7" y="20.574" smashed="yes" rot="MR0"/>
+<element name="LOGO1" library="SparkFun-Aesthetics" package="SFE_LOGO_NAME_FLAME_.1" value="SFE_LOGO_NAME_FLAME.1_INCH" x="12.7" y="12" smashed="yes" rot="MR0"/>
 <element name="LOGO2" library="SparkFun-Aesthetics" package="OSHW-LOGO-S" value="OSHW-LOGOS" x="23.495" y="23.495" smashed="yes" rot="MR0"/>
 <element name="U$18" library="buzzard_labels (2)" package="EVI1" value="" x="11" y="15.6" smashed="yes"/>
 <element name="U$19" library="buzzard_labels (2)" package="I2C0" value="" x="11.1" y="8.3" smashed="yes"/>
 <element name="U$20" library="buzzard_labels (3)" package="LED2" value="" x="6.29" y="7" smashed="yes" rot="MR0"/>
-<element name="U$21" library="buzzard_labels (4)" package="QWIIC_RTC0" value="" x="17" y="18.4" smashed="yes" rot="MR0"/>
-<element name="U$22" library="buzzard_labels (4)" package="_RV#88031" value="" x="17" y="17.1" smashed="yes" rot="MR0"/>
+<element name="U$21" library="buzzard_labels (4)" package="QWIIC_RTC0" value="" x="17" y="9.51" smashed="yes" rot="MR0"/>
+<element name="U$22" library="buzzard_labels (4)" package="_RV#88031" value="" x="17" y="8.21" smashed="yes" rot="MR0"/>
 <element name="FD1" library="SparkFun-Aesthetics" package="FIDUCIAL-MICRO" value="FIDUCIALUFIDUCIAL" x="2.54" y="6.35" smashed="yes"/>
 <element name="FD2" library="SparkFun-Aesthetics" package="FIDUCIAL-MICRO" value="FIDUCIALUFIDUCIAL" x="2.54" y="6.35" smashed="yes" rot="MR0"/>

Commit message: adding resistor on OE line
Parts:
- added R6: 100k, SparkFun-Resistors:0603
Connections:
- net CLKOE: now also R6.2
- net GND: now also R6.1
Routing:
- net CLKOE: track 14.7 -> 17.3 mm
Other:
- board text added: "v11"
- board text removed: "v10"
Changed lines of the file:
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@@
 <wire x1="25.4" y1="25.4" x2="0" y2="25.4" width="0.2032" layer="20"/>
 <wire x1="0" y1="25.4" x2="0" y2="0" width="0.2032" layer="20"/>
-<text x="1.6" y="3.2" size="1.27" layer="16" font="vector" ratio="15" rot="MR270">v10</text>
+<text x="1.6" y="3.2" size="1.27" layer="16" font="vector" ratio="15" rot="MR270">v11</text>
 <dimension x1="0" y1="0" x2="0" y2="25.4" x3="-2.54" y3="12.7" textsize="1.016" textratio="15" layer="47" unit="inch"/>
 <dimension x1="0" y1="25.4" x2="25.4" y2="25.4" x3="12.7" y3="27.94" textsize="1.016" textratio="15" layer="47" unit="inch"/>
@@
 <element name="U$24" library="buzzard_labels (4)" package="_RV#88031" value="" x="-0.49" y="17.79" smashed="yes"/>
 <element name="U$25" library="buzzard_labels (5)" package="RTC0" value="" x="1.47" y="19.05" smashed="yes"/>
+<element name="R6" library="SparkFun-Resistors" package="0603" value="100k" x="24.13" y="3.81" smashed="yes" rot="R270">
+<attribute name="NAME" x="24.892" y="3.81" size="0.6096" layer="25" font="vector" ratio="20" rot="R270" align="bottom-center"/>
+<attribute name="PROD_ID" value="RES-07828" x="24.13" y="3.81" size="1.778" layer="27" rot="R270" display="off"/>
+<attribute name="VALUE" x="23.368" y="3.81" size="0.6096" layer="27" font="vector" ratio="20" rot="R270" align="top-center"/>
+</element>
 </elements>
 <signals>
@@
 <via x="23.6228" y="7.7508" extent="1-16" drill="0.381"/>
 <via x="21.6228" y="16.7508" extent="1-16" drill="0.381"/>
+<contactref element="R6" pad="1"/>
 </signal>
 <signal name="SCL">
@@
 <contactref element="U1" pad="4"/>
 <contactref element="J3" pad="8"/>
-<wire x1="21.59" y1="1.27" x2="21.59" y2="5.715" width="0.2032" layer="1"/>
+<wire x1="21.59" y1="1.27" x2="21.59" y2="3" width="0.2032" layer="1"/>
+<wire x1="21.59" y1="3" x2="21.59" y2="5.715" width="0.2032" layer="1"/>
 <wire x1="21.59" y1="5.715" x2="19.05" y2="8.255" width="0.2032" layer="1"/>
 <wire x1="16.51" y1="8.255" x2="16.1925" y2="8.5725" width="0.2032" layer="1"/>
@@
 <wire x1="15.8178" y1="9.9822" x2="14.5415" y2="9.9822" width="0.2032" layer="1"/>
 <wire x1="16.1925" y1="9.6075" x2="15.8178" y2="9.9822" width="0.2032" layer="1"/>
+<contactref element="R6" pad="2"/>
+<wire x1="24.13" y1="2.96" x2="21.63" y2="2.96" width="0.1778" layer="1"/>
+<wire x1="21.63" y1="2.96" x2="21.59" y2="3" width="0.1778" layer="1"/>
 </signal>
 <signal name="!EVI">
